File: 2.0.kicad_sch (KiCad schematic)
At the start: 26 parts, among them U1 BAT-HLD-001-TR

Commit message: Fixed PCB
Parts:
- removed U1: BAT-HLD-001-TR, BATHLD001TR, symbol BAT-HLD-001-TR:BAT-HLD-001-TR
- added J1: MK-12C02, user-footprints:MK12C02, symbol MK-12C02:MK-12C02
- BT1: footprint BC-2001:BC2001 -> user-footprints:CR2032_holder_ali
Connections:
- net at BT1.1 (+): now also J1.2 (COM)
- net at D1.2 (A), D10.2 (A), D11.2 (A)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: now also J1.3 (NO)
Changed lines of the file:
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@@
     (stroke (width 0) (type default) (color 0 0 0 0))
   )
-  (wire (pts (xy 48.26 86.36) (xy 48.26 88.9))
+  (wire (pts (xy 48.26 82.55) (xy 48.26 88.9))
+    (stroke (width 0) (type default) (color 0 0 0 0))
+  )
+  (wire (pts (xy 45.72 82.55) (xy 45.72 86.36))
     (stroke (width 0) (type default) (color 0 0 0 0))
   )
@@
       (effects (font (size 1.27 1.27)) (justify left))
     )
-    (property "Footprint" "BC-2001:BC2001" (id 2) (at 38.1 94.996 90)
+    (property "Footprint" "user-footprints:CR2032_holder_ali" (id 2) (at 38.1 94.996 90)
       (effects (font (size 1.27 1.27)) hide)
     )
@@
     (pin "1")
     (pin "2")
-  )
-  (symbol (lib_id "BAT-HLD-001-TR:BAT-HLD-001-TR") (at 45.72 86.36 90) (unit 1)
-    (in_bom yes) (on_board yes)
-    (property "Reference" "U1" (id 0) (at 54.0512 77.7748 90)
-      (effects (font (size 1.27 1.27)) (justify right))
-    )
-    (property "Value" "BAT-HLD-001-TR" (id 1) (at 54.0512 80.0862 90)
-      (effects (font (size 1.27 1.27)) (justify right))
-    )
-    (property "Footprint" "BATHLD001TR" (id 2) (at 43.18 69.85 0)
-      (effects (font (size 1.27 1.27)) (justify left) hide)
-    )
-    (property "Datasheet" "https://datasheet.datasheetarchive.com/originals/distributors/DKDS-31/603271.pdf" (id 3) (at 45.72 69.85 0)
-      (effects (font (size 1.27 1.27)) (justify left) hide)
-    )
-    (property "Description" "Coin Cell Battery Holders Linx CR2032 Battery Holder, Tape n Reel" (id 4) (at 48.26 69.85 0)
-      (effects (font (size 1.27 1.27)) (justify left) hide)
-    )
-    (property "Height" "4.2" (id 5) (at 50.8 69.85 0)
-      (effects (font (size 1.27 1.27)) (justify left) hide)
-    )
-    (property "Manufacturer_Name" "Linx Technologies" (id 6) (at 53.34 69.85 0)
-      (effects (font (size 1.27 1.27)) (justify left) hide)
-    )
-    (property "Manufacturer_Part_Number" "BAT-HLD-001-TR" (id 7) (at 55.88 69.85 0)
-      (effects (font (size 1.27 1.27)) (justify left) hide)
-    )
-    (property "Mouser Part Number" "712-BAT-HLD-001-TR" (id 8) (at 58.42 69.85 0)
-      (effects (font (size 1.27 1.27)) (justify left) hide)
-    )
-    (property "Mouser Price/Stock" "https://www.mouser.co.uk/ProductDetail/Linx-Technologies/BAT-HLD-001-TR?qs=K5ta8V%252BWhtZh3MyWmkkmjQ%3D%3D" (id 9) (at 60.96 69.85 0)
-      (effects (font (size 1.27 1.27)) (justify left) hide)
-    )
-    (property "Arrow Part Number" "" (id 10) (at 63.5 69.85 0)
-      (effects (font (size 1.27 1.27)) (justify left) hide)
-    )
-    (property "Arrow Price/Stock" "" (id 11) (at 66.04 69.85 0)
-      (effects (font (size 1.27 1.27)) (justify left) hide)
-    )
-    (pin "1")
-    (pin "2")
-    (pin "3")
   )
   (symbol (lib_id "power:GND") (at 38.1 107.95 0) (unit 1)
@@
     )
     (pin "1")
+  )
+  (symbol (lib_id "MK-12C02:MK-12C02") (at 43.18 82.55 90) (unit 1)
+    (in_bom yes) (on_board yes) (fields_autoplaced)
+    (property "Reference" "J1" (id 0) (at 54.0512 68.9415 90)
+      (effects (font (size 1.27 1.27)) (justify right))
+    )
+    (property "Value" "MK-12C02" (id 1) (at 54.0512 71.7166 90)
+      (effects (font (size 1.27 1.27)) (justify right))
+    )
+    (property "Footprint" "user-footprints:MK12C02" (id 2) (at 40.64 60.96 0)
+      (effects (font (size 1.27 1.27)) (justify left) hide)
+    )
+    (property "Datasheet" "https://statics3.seeedstudio.com/images/opl/datasheet/311030001.pdf" (id 3) (at 43.18 60.96 0)
+      (effects (font (size 1.27 1.27)) (justify left) hide)
+    )
+    (property "Description" "connector" (id 4) (at 45.72 60.96 0)
+      (effects (font (size 1.27 1.27)) (justify left) hide)
+    )
+    (property "Height" "3.3" (id 5) (at 48.26 60.96 0)
+      (effects (font (size 1.27 1.27)) (justify left) hide)
+    )
+    (property "Manufacturer_Name" "XIEJIA ELECTRONICS" (id 6) (at 50.8 60.96 0)
+      (effects (font (size 1.27 1.27)) (justify left) hide)
+    )
+    (property "Manufacturer_Part_Number" "MK-12C02" (id 7) (at 53.34 60.96 0)
+      (effects (font (size 1.27 1.27)) (justify left) hide)
+    )
+    (property "Mouser Part Number" "" (id 8) (at 55.88 60.96 0)
+      (effects (font (size 1.27 1.27)) (justify left) hide)
+    )
+    (property "Mouser Price/Stock" "" (id 9) (at 58.42 60.96 0)
+      (effects (font (size 1.27 1.27)) (justify left) hide)
+    )
+    (property "Arrow Part Number" "" (id 10) (at 60.96 60.96 0)
+      (effects (font (size 1.27 1.27)) (justify left) hide)
+    )
+    (property "Arrow Price/Stock" "" (id 11) (at 63.5 60.96 0)
+      (effects (font (size 1.27 1.27)) (justify left) hide)
+    )
+    (pin "1")
+    (pin "2")
+    (pin "3")
+    (pin "MP1")
+    (pin "MP2")
+    (pin "MP3")
+    (pin "MP4")
   )
   (sheet_instances
@@
     )
     (path "/00000000-0000-0000-0000-000061c2ebf8"
-      (reference "BT1") (unit 1) (value "Battery_Cell") (footprint "BC-2001:BC2001")
+      (reference "BT1") (unit 1) (value "Battery_Cell") (footprint "user-footprints:CR2032_holder_ali")
     )
     (path "/00000000-0000-0000-0000-000061c30ea3"
@@
       (reference "D12") (unit 1) (value "LED") (footprint "LED_SMD:LED_0805_2012Metric_Pad1.15x1.40mm_HandSolder")
     )
+    (path "/ffb86135-b43f-4a42-9aa6-73aa7ba972a9"
+      (reference "J1") (unit 1) (value "MK-12C02") (footprint "user-footprints:MK12C02")
+    )
     (path "/00000000-0000-0000-0000-000061c376f8"
       (reference "R1") (unit 1) (value "1k") (footprint "Resistor_SMD:R_0805_2012Metric_Pad1.20x1.40mm_HandSolder")
@@
       (reference "R12") (unit 1) (value "1k") (footprint "Resistor_SMD:R_0805_2012Metric_Pad1.20x1.40mm_HandSolder")
     )
-    (path "/00000000-0000-0000-0000-000061c3a16a"
-      (reference "U1") (unit 1) (value "BAT-HLD-001-TR") (footprint "BATHLD001TR")
-    )
-  )
+  )
