File: 2.0.kicad_pcb (KiCad board)
At the start: 2 copper layers, 38.1 x 50 mm, 26 parts, among them J1 MK-12C02

Commit message: Fixed position ordernr
Other:
- board text added: "JLCJLCJLCJLC"
Changed lines of the file:
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@@
     (property "Sheetname" "")
     (attr through_hole)
-    (fp_text reference "J1" (at 0 0.575 65) (layer "B.SilkS")
+    (fp_text reference "J1" (at 0 0.575 65) (layer "B.SilkS") hide
       (effects (font (size 1.27 1.27) (thickness 0.254)) (justify mirror))
     )
@@
     (property "Sheetname" "")
     (attr smd)
-    (fp_text reference "BT1" (at 0 12.7 unlocked) (layer "B.SilkS")
+    (fp_text reference "BT1" (at 0 12.7 unlocked) (layer "B.SilkS") hide
       (effects (font (size 1 1) (thickness 0.15)) (justify mirror))
     )
-    (fp_text value "Battery_Cell" (at 0 -12.7 unlocked) (layer "B.Fab")
+    (fp_text value "Battery_Cell" (at 0 -12.7 unlocked) (layer "B.Fab") hide
       (effects (font (size 1 1) (thickness 0.15)) (justify mirror))
     )
@@
     (effects (font (size 1 1) (thickness 0.15)) (justify mirror))
   )
+  (gr_text "JLCJLCJLCJLC" (at 168.3 120.89) (layer "B.SilkS")
+    (effects (font (size 0.9 0.9) (thickness 0.15)) (justify mirror))
+  )
   (gr_text "https://github.com/gjlp25/KiCad_FlashyTree" (at 184.51 96.6 -67) (layer "B.SilkS")
